File: V2/v2/southpawcase v2/southpawcase.kicad_pcb (KiCad board)
At the start: 2 copper layers, 391.2 x 109.5 mm, 4 parts

Commit message: fixed logo changed files added compat, ordered protos
Parts:
- removed the G*** at (188.1, 54.8) (x2)
- added G***: LOGO, drewkeys:v2, F.Cu at (45.1, 104.4)
- added G***: LOGO, drewkeys:paw paw, F.Cu at (188.1, 54.8)
- moved G*** 15.0 mm to (26.2, 104.8) (x2)
Other:
- board size 391.2 x 109.5 mm -> 391.3 x 109.5 mm
