File: V2/v2/southpawplate v2/southpawplate.kicad_pcb (KiCad board)
At the start: 2 copper layers, 391.2 x 109.5 mm, 4 parts

Commit message: fixed logo changed files added compat, ordered protos
Parts:
- added G***: LOGO, drewkeys:v2, B.Cu at (331.2, 104.5)
- added G***: LOGO, drewkeys:v2, F.Cu at (27.5, 104.4)
Changed lines of the file:
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@@
     (tracks 0)
     (zones 0)
-    (modules 4)
+    (modules 6)
     (nets 1)
   )
@@
     (uvia_drill 0.1)
   )
+  (module drewkeys:v2 (layer B.Cu)
+    (at 331.2 104.5 180)
+    (fp_text reference G*** (at 0 0) (layer B.SilkS) hide
+      (effects (font (size 1.524 1.524) (thickness 0.3)) (justify mirror))
+    )
+    (fp_text value LOGO (at 0.75 0) (layer B.SilkS) hide
+      (effects (font (size 1.524 1.524) (thickness 0.3)) (justify mirror))
+    )
+    (fp_poly (pts (xy -2.8321 1.106375) (xy -2.159 1.0922) (xy -2.032 0) (xy -1.992882 -0.319201)
+      (xy -1.954542 -0.600753) (xy -1.919256 -0.830279) (xy -1.889301 -0.993401) (xy -1.866953 -1.075743)
+      (xy -1.860545 -1.082821) (xy -1.825563 -1.037007) (xy -1.751087 -0.913343) (xy -1.644099 -0.724324)
+      (xy -1.511581 -0.482446) (xy -1.360515 -0.200204) (xy -1.250247 0.009379) (xy -0.684404 1.0922)
+      (xy -0.494602 1.0922) (xy -0.368543 1.086007) (xy -0.296859 1.070687) (xy -0.2921 1.066394)
+      (xy -0.312365 1.017355) (xy -0.375584 0.888689) (xy -0.476636 0.690274) (xy -0.610399 0.431991)
+      (xy -0.771751 0.123717) (xy -0.95557 -0.22467) (xy -1.156735 -0.603289) (xy -1.1938 -0.672781)
+      (xy -2.1082 -2.386149) (xy -2.551733 -2.386874) (xy -2.765324 -2.385549) (xy -2.898307 -2.377331)
+      (xy -2.971656 -2.357141) (xy -3.006348 -2.319897) (xy -3.020609 -2.2733) (xy -3.034036 -2.195789)
+      (xy -3.05924 -2.034646) (xy -3.094087 -1.804592) (xy -3.136442 -1.520345) (xy -3.18417 -1.196628)
+      (xy -3.235138 -0.848158) (xy -3.287211 -0.489658) (xy -3.338254 -0.135846) (xy -3.386132 0.198556)
+      (xy -3.428712 0.498829) (xy -3.463859 0.750253) (xy -3.489439 0.938108) (xy -3.503316 1.047672)
+      (xy -3.5052 1.068642) (xy -3.455422 1.090998) (xy -3.309464 1.104602) (xy -3.072394 1.10917)
+      (xy -2.8321 1.106375)) (layer B.SilkS) (width 0.01))
+    (fp_poly (pts (xy 2.432012 2.356089) (xy 2.72102 2.301643) (xy 2.907703 2.236595) (xy 3.129634 2.098568)
+      (xy 3.328292 1.915657) (xy 3.472772 1.718438) (xy 3.508602 1.64205) (xy 3.550386 1.430411)
+      (xy 3.544462 1.176887) (xy 3.493886 0.927599) (xy 3.454249 0.822109) (xy 3.305559 0.580582)
+      (xy 3.062733 0.304059) (xy 2.725528 -0.007687) (xy 2.2937 -0.354888) (xy 1.885767 -0.654201)
+      (xy 1.053734 -1.2446) (xy 2.043279 -1.258348) (xy 3.032824 -1.272097) (xy 2.923909 -1.817148)
+      (xy 2.814994 -2.3622) (xy 1.046207 -2.375564) (xy 0.567937 -2.378655) (xy 0.182195 -2.379759)
+      (xy -0.120078 -2.378579) (xy -0.34794 -2.374818) (xy -0.510449 -2.368181) (xy -0.616664 -2.35837)
+      (xy -0.675643 -2.345089) (xy -0.696445 -2.328042) (xy -0.695577 -2.318559) (xy -0.67239 -2.228796)
+      (xy -0.644389 -2.081443) (xy -0.631504 -2.000992) (xy -0.616372 -1.909995) (xy -0.594837 -1.832161)
+      (xy -0.557204 -1.756872) (xy -0.493778 -1.67351) (xy -0.394862 -1.571456) (xy -0.250761 -1.440092)
+      (xy -0.051778 -1.268798) (xy 0.211782 -1.046956) (xy 0.3302 -0.947767) (xy 0.705604 -0.630883)
+      (xy 1.012667 -0.365524) (xy 1.26322 -0.140807) (xy 1.469095 0.054151) (xy 1.642124 0.230235)
+      (xy 1.794137 0.398327) (xy 1.796271 0.400789) (xy 2.004808 0.665887) (xy 2.139449 0.903215)
+      (xy 2.211955 1.139639) (xy 2.234084 1.400845) (xy 2.228312 1.585331) (xy 2.202651 1.703391)
+      (xy 2.147067 1.789722) (xy 2.111128 1.82605) (xy 2.028618 1.890543) (xy 1.935858 1.922297)
+      (xy 1.799038 1.92858) (xy 1.664466 1.922068) (xy 1.388042 1.879158) (xy 1.178108 1.780274)
+      (xy 1.011412 1.609549) (xy 0.882651 1.388573) (xy 0.800695 1.192486) (xy 0.751153 0.990194)
+      (xy 0.724273 0.7388) (xy 0.720591 0.675668) (xy 0.701984 0.440944) (xy 0.675905 0.306102)
+      (xy 0.642068 0.269676) (xy 0.641175 0.269992) (xy 0.563537 0.292257) (xy 0.421075 0.32744)
+      (xy 0.28595 0.358583) (xy -0.012299 0.42532) (xy 0.011901 0.763541) (xy 0.076509 1.125136)
+      (xy 0.209333 1.475687) (xy 0.394836 1.775551) (xy 0.421069 1.807631) (xy 0.596415 1.963578)
+      (xy 0.841267 2.113197) (xy 1.124004 2.240343) (xy 1.413009 2.328872) (xy 1.462221 2.339259)
+      (xy 1.769937 2.377218) (xy 2.104093 2.382054) (xy 2.432012 2.356089)) (layer B.SilkS) (width 0.01))
+  )
+  (module drewkeys:v2 (layer F.Cu)
+    (at 27.5 104.4)
+    (fp_text reference G*** (at 0 0) (layer F.SilkS) hide
+      (effects (font (size 1.524 1.524) (thickness 0.3)))
+    )
+    (fp_text value LOGO (at 0.75 0) (layer F.SilkS) hide
+      (effects (font (size 1.524 1.524) (thickness 0.3)))
+    )
+    (fp_poly (pts (xy 2.432012 -2.356089) (xy 2.72102 -2.301643) (xy 2.907703 -2.236595) (xy 3.129634 -2.098568)
+      (xy 3.328292 -1.915657) (xy 3.472772 -1.718438) (xy 3.508602 -1.64205) (xy 3.550386 -1.430411)
+      (xy 3.544462 -1.176887) (xy 3.493886 -0.927599) (xy 3.454249 -0.822109) (xy 3.305559 -0.580582)
+      (xy 3.062733 -0.304059) (xy 2.725528 0.007687) (xy 2.2937 0.354888) (xy 1.885767 0.654201)
+      (xy 1.053734 1.2446) (xy 2.043279 1.258348) (xy 3.032824 1.272097) (xy 2.923909 1.817148)
+      (xy 2.814994 2.3622) (xy 1.046207 2.375564) (xy 0.567937 2.378655) (xy 0.182195 2.379759)
+      (xy -0.120078 2.378579) (xy -0.34794 2.374818) (xy -0.510449 2.368181) (xy -0.616664 2.35837)
+      (xy -0.675643 2.345089) (xy -0.696445 2.328042) (xy -0.695577 2.318559) (xy -0.67239 2.228796)
+      (xy -0.644389 2.081443) (xy -0.631504 2.000992) (xy -0.616372 1.909995) (xy -0.594837 1.832161)
+      (xy -0.557204 1.756872) (xy -0.493778 1.67351) (xy -0.394862 1.571456) (xy -0.250761 1.440092)
+      (xy -0.051778 1.268798) (xy 0.211782 1.046956) (xy 0.3302 0.947767) (xy 0.705604 0.630883)
+      (xy 1.012667 0.365524) (xy 1.26322 0.140807) (xy 1.469095 -0.054151) (xy 1.642124 -0.230235)
+      (xy 1.794137 -0.398327) (xy 1.796271 -0.400789) (xy 2.004808 -0.665887) (xy 2.139449 -0.903215)
+      (xy 2.211955 -1.139639) (xy 2.234084 -1.400845) (xy 2.228312 -1.585331) (xy 2.202651 -1.703391)
+      (xy 2.147067 -1.789722) (xy 2.111128 -1.82605) (xy 2.028618 -1.890543) (xy 1.935858 -1.922297)
+      (xy 1.799038 -1.92858) (xy 1.664466 -1.922068) (xy 1.388042 -1.879158) (xy 1.178108 -1.780274)
+      (xy 1.011412 -1.609549) (xy 0.882651 -1.388573) (xy 0.800695 -1.192486) (xy 0.751153 -0.990194)
+      (xy 0.724273 -0.7388) (xy 0.720591 -0.675668) (xy 0.701984 -0.440944) (xy 0.675905 -0.306102)
+      (xy 0.642068 -0.269676) (xy 0.641175 -0.269992) (xy 0.563537 -0.292257) (xy 0.421075 -0.32744)
+      (xy 0.28595 -0.358583) (xy -0.012299 -0.42532) (xy 0.011901 -0.763541) (xy 0.076509 -1.125136)
+      (xy 0.209333 -1.475687) (xy 0.394836 -1.775551) (xy 0.421069 -1.807631) (xy 0.596415 -1.963578)
+      (xy 0.841267 -2.113197) (xy 1.124004 -2.240343) (xy 1.413009 -2.328872) (xy 1.462221 -2.339259)
+      (xy 1.769937 -2.377218) (xy 2.104093 -2.382054) (xy 2.432012 -2.356089)) (layer F.SilkS) (width 0.01))
+    (fp_poly (pts (xy -2.8321 -1.106375) (xy -2.159 -1.0922) (xy -2.032 0) (xy -1.992882 0.319201)
+      (xy -1.954542 0.600753) (xy -1.919256 0.830279) (xy -1.889301 0.993401) (xy -1.866953 1.075743)
+      (xy -1.860545 1.082821) (xy -1.825563 1.037007) (xy -1.751087 0.913343) (xy -1.644099 0.724324)
+      (xy -1.511581 0.482446) (xy -1.360515 0.200204) (xy -1.250247 -0.009379) (xy -0.684404 -1.0922)
+      (xy -0.494602 -1.0922) (xy -0.368543 -1.086007) (xy -0.296859 -1.070687) (xy -0.2921 -1.066394)
+      (xy -0.312365 -1.017355) (xy -0.375584 -0.888689) (xy -0.476636 -0.690274) (xy -0.610399 -0.431991)
+      (xy -0.771751 -0.123717) (xy -0.95557 0.22467) (xy -1.156735 0.603289) (xy -1.1938 0.672781)
+      (xy -2.1082 2.386149) (xy -2.551733 2.386874) (xy -2.765324 2.385549) (xy -2.898307 2.377331)
+      (xy -2.971656 2.357141) (xy -3.006348 2.319897) (xy -3.020609 2.2733) (xy -3.034036 2.195789)
+      (xy -3.05924 2.034646) (xy -3.094087 1.804592) (xy -3.136442 1.520345) (xy -3.18417 1.196628)
+      (xy -3.235138 0.848158) (xy -3.287211 0.489658) (xy -3.338254 0.135846) (xy -3.386132 -0.198556)
+      (xy -3.428712 -0.498829) (xy -3.463859 -0.750253) (xy -3.489439 -0.938108) (xy -3.503316 -1.047672)
+      (xy -3.5052 -1.068642) (xy -3.455422 -1.090998) (xy -3.309464 -1.104602) (xy -3.072394 -1.10917)
+      (xy -2.8321 -1.106375)) (layer F.SilkS) (width 0.01))
+  )
   (module Logos:southpaw75small (layer B.Cu)
